Commit message: update object urdf

File: assets/objects/urdf/cylinder_3.urdf (robot description, URDF)
Before this commit: robot cylinder_3, 2 links, 1 joints
Joints:
- joint world_to_indenter: origin xyz=0.0 0.0 0.0 rpy=0.0 0.0 0.0 -> xyz=0.0 -0.001 0.0 rpy=0.0 0.0 0.0

File: assets/objects/urdf/nut.urdf (robot description, URDF)
Before this commit: robot nut, 2 links, 1 joints
Joints:
- joint world_to_indenter: origin xyz=0.0 0.0 0.0 rpy=0.0 0.0 0.0 -> xyz=0.0 -0.0026 0.0 rpy=0.0 0.0 0.0

File: assets/objects/urdf/sphere_3.urdf (robot description, URDF)
Before this commit: robot sphere_3, 2 links, 1 joints
Joints:
- joint world_to_indenter: origin xyz=0.0 0.0 0.0 rpy=0.0 0.0 0.0 -> xyz=0.0 -0.002 0.0 rpy=0.0 0.0 0.0
